File: Bluetooth_5.sch (KiCad schematic (older format))
At the start: 39 parts

Commit message: added datasheet and oscillator Crystal Hz
Parts:
- renumbered SR_H71 to 38.4Mhz_SR_H71
Changed lines of the file:
@@
 	5550 3900 5550 3950
 $Comp
-L Crystal_resonators:HC_49S SR_H71
+L Crystal_resonators:HC_49S 38.4Mhz_SR_H71
 U 1 1 5CEA37F1
 P 5800 4450
-F 0 "SR_H71" H 5800 4150 50  0000 C CNN
+F 0 "38.4Mhz_SR_H71" H 5800 4150 50  0000 C CNN
 F 1 "HC_49S" H 5800 4300 50  0000 C CNN
 F 2 "Crystal_resonators:HC_49S" H 5750 4600 50  0001 C CNN
